File: DucMinh.kicad_pcb (KiCad board)
At the start: 2 copper layers, 95.3 x 48.1 mm, 66 parts, among them J1 Power, J10 HC05, J11 PWR_Selection, J12 BOOT0, J2 M1, J3 USB_B_Micro, J4 M2, J5 M3, J6 AS5600, J7 STLink, J8 Stepper_Motor, J9 STLink_EN, SW1 SW_Push, U10 BTS7960B, U2 AMS1117-3.3, U3 LM2596SX-5.0/NOPB, U4 TMC2209_SILENTSTEPSTICK, U5 BTS7960B, U6 STM32F103RCT6, U8 BTS7960B, Y1 8 MHz

Commit message: final
Parts:
- removed J9: STLink_EN, Connector_PinHeader_2.54mm:PinHeader_1x02_P2.54mm_Vertical
- removed R29, R31, R33: 10k, Resistor_SMD:R_0603_1608Metric_Pad0.98x0.95mm_HandSolder
- moved Y1 108.8 mm to (81.2, 110.5), turned to 180 degrees
- moved C15 108.4 mm to (74.3, 106.9), turned to 180 degrees
- moved C14 100.6 mm to (83.1, 106.9)
- moved DS1 100.5 mm to (92.7, 90.5), turned to 45 degrees
- moved D1 98.9 mm to (84.7, 58.8), turned to 180 degrees
- moved C9 98.8 mm to (87.2, 110.7), turned to -90 degrees
- moved R3 91.6 mm to (90.7, 105.9)
- moved DS2 90.7 mm to (102.5, 95.3), turned to 135 degrees
- moved R7 90.1 mm to (95.3, 90.2), turned to 45 degrees
- moved SW1 88.0 mm to (89.8, 108.5)
- moved C18 87.5 mm to (100.9, 81.7), turned to -135 degrees
- moved DS4 86.6 mm to (111.9, 67.2), turned to 180 degrees
- moved C10 86.3 mm to (97.8, 89.9), turned to 135 degrees
- moved R16 83.4 mm to (101.4, 96.5), turned to 135 degrees
- moved FB1 81.7 mm to (108.3, 100.8), turned to -45 degrees
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Connections:
- J7 pad 1: 3V3_STLINK -> unconnected-(J7-Pin_1-Pad1)
- U10 pad 3: Net-(U10-INH) -> +3V3
- U5 pad 3: Net-(U5-INH) -> +3V3
- U6 pad 29: unconnected-(U6-PB10-Pad29) -> TX2
- U6 pad 30: unconnected-(U6-PB11-Pad30) -> RX2
- U6 pad 33: unconnected-(U6-PB12-Pad33) -> DIR_PIN
- U6 pad 34: unconnected-(U6-PB13-Pad34) -> STEP_PIN
- U6 pad 35: unconnected-(U6-PB14-Pad35) -> MS2_PIN
- U6 pad 36: unconnected-(U6-PB15-Pad36) -> MS1_PIN
- U6 pad 37: unconnected-(U6-PC6-Pad37) -> ENABLE_PIN
- U6 pad 55: unconnected-(U6-PB3-Pad55) -> PWM1
- U6 pad 56: unconnected-(U6-PB4-Pad56) -> PWM2
- U6 pad 57: unconnected-(U6-PB5-Pad57) -> PWM3
- U6 pad 58: unconnected-(U6-PB6-Pad58) -> SCL2
- U6 pad 59: unconnected-(U6-PB7-Pad59) -> SDA2
- U8 pad 3: Net-(U8-INH) -> +3V3
Routing:
- net +3V3: track 0.00 -> 250.6 mm, vias 0 -> 4
- net GND: track 7.60 -> 64.1 mm, vias 56 -> 74
- net PWM1: track 1.27 -> 45.6 mm, vias 1 -> 2
- net Net-(U6-PD0-OSC_IN): track 0.00 -> 40.3 mm, vias 0 -> 2
- net PWM3: track 1.27 -> 41.4 mm, vias 1 -> 2
- net PWM2: track 1.27 -> 39.6 mm, vias 1 -> 2
- net DIR_PIN: track 0.00 -> 37.0 mm, vias 0 -> 2
- net STEP_PIN: track 0.00 -> 35.8 mm, vias 0 -> 2
- net RESET: track 0.00 -> 34.1 mm, vias 0 -> 2
- net Net-(U6-PD1_OSC_OUT): track 0.00 -> 34.0 mm, vias 0 -> 2
- net ENABLE_PIN: track 0.00 -> 32.6 mm, vias 0 -> 2
- net MS1_PIN: track 0.00 -> 32.6 mm, vias 0 -> 2
- net MS2_PIN: track 0.00 -> 32.4 mm, vias 0 -> 2
- net SCL2: track 0.00 -> 27.4 mm, vias 0 -> 1
- net SDA2: track 0.00 -> 25.1 mm, vias 0 -> 1
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- added copper zone on F.Cu, net 5V_LDO
- added copper zone on B.Cu, net M1+
- added copper zone on B.Cu, net M2+
- added copper zone on B.Cu, net M3+
- added copper zone on F.Cu, net Net-(D2-A)
Other:
- board size 95.3 x 48.1 mm -> 90 x 80 mm
- board text added: "+"
- board text added: "-"
- board text added: "0"
- board text added: "1"
- board text added: "3V3"
- board text added: "4xM3"
- board text added: "6-24VDC"
- board text added: "A+"
- board text added: "A-"
- board text added: "AS5600"
- board text added: "B+"
- board text added: "B-"
- board text added: "BOOT0"
- board text added: "GND"
- board text added: "HC05"
- board text added: "RESET"
- board text added: "RX"
- board text added: "SCL"
- board text added: "SDA"
- board text added: "STLINK"
- board text added: "SWCLK"
- board text added: "SWDIO"
- board text added: "TX"
- board text added: "VIN"
- board text added: "VUSB"

Commit message: final2
Connections:
- U6 pad 33: DIR_PIN -> unconnected-(U6-PB12-Pad33)
- U6 pad 34: STEP_PIN -> unconnected-(U6-PB13-Pad34)
- U6 pad 35: MS2_PIN -> unconnected-(U6-PB14-Pad35)
- U6 pad 36: MS1_PIN -> unconnected-(U6-PB15-Pad36)
- U6 pad 37: ENABLE_PIN -> unconnected-(U6-PC6-Pad37)
- U6 pad 39: unconnected-(U6-PC8-Pad39) -> DIR_PIN
- U6 pad 40: unconnected-(U6-PC9-Pad40) -> STEP_PIN
- U6 pad 41: unconnected-(U6-PA8-Pad41) -> MS2_PIN
- U6 pad 42: unconnected-(U6-PA9-Pad42) -> MS1_PIN
- U6 pad 43: unconnected-(U6-PA10-Pad43) -> ENABLE_PIN
Routing:
- net ENABLE_PIN: track 32.6 -> 31.6 mm
- net MS1_PIN: track 32.6 -> 31.7 mm
- net MS2_PIN: track 32.4 -> 31.7 mm
- net STEP_PIN: track 35.8 -> 35.1 mm

Commit message: update apperance
Other:
- board text added: "VBUS"
- board text removed: "4xM3"
- board text removed: "VUSB"
Changed lines of the file:
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@@
 		)
 	)
-	(gr_line
-		(start 46.81 45.38)
-		(end 47.56 46.13)
+	(gr_circle
+		(center 46.81 42.4)
+		(end 48.81 42.4)
 		(stroke
-			(width 0.1)
-			(type default)
+			(width 0.7)
+			(type solid)
 		)
+		(fill no)
 		(layer "F.SilkS")
 	)
-	(gr_line
-		(start 46.06 46.13)
-		(end 46.81 45.38)
+	(gr_circle
+		(center 106.81 114.4)
+		(end 109.51 114.4)
 		(stroke
-			(width 0.1)
-			(type default)
+			(width 0.2)
+			(type solid)
+		)
+		(fill no)
+		(layer "F.SilkS")
+	)
+	(gr_circle
+		(center 46.81 114.4)
+		(end 49.51 114.4)
+		(stroke
+			(width 0.2)
+			(type solid)
 		)
+		(fill no)
 		(layer "F.SilkS")
 	)
@@
 		(layer "F.SilkS")
 	)
+	(gr_circle
+		(center 46.81 42.4)
+		(end 49.51 42.4)
+		(stroke
+			(width 0.2)
+			(type solid)
+		)
+		(fill no)
+		(layer "F.SilkS")
+	)
 	(gr_line
 		(start 104.42 80.13)
@@
 		(layer "F.SilkS")
 	)
-	(gr_line
-		(start 46.810001 49.29)
-		(end 46.81 45.38)
+	(gr_circle
+		(center 106.81 114.4)
+		(end 108.81 114.4)
 		(stroke
-			(width 0.1)
-			(type default)
+			(width 0.7)
+			(type solid)
+		)
+		(fill no)
+		(layer "F.SilkS")
+	)
+	(gr_circle
+		(center 46.81 114.4)
+		(end 48.81 114.4)
+		(stroke
+			(width 0.7)
+			(type solid)
+		)
+		(fill no)
+		(layer "F.SilkS")
+	)
+	(gr_circle
+		(center 106.81 42.4)
+		(end 109.51 42.4)
+		(stroke
+			(width 0.2)
+			(type solid)
 		)
+		(fill no)
+		(layer "F.SilkS")
+	)
+	(gr_circle
+		(center 106.81 42.4)
+		(end 108.81 42.4)
+		(stroke
+			(width 0.7)
+			(type solid)
+		)
+		(fill no)
 		(layer "F.SilkS")
 	)
@@
 	)
 	(gr_circle
+		(center 106.81 42.4)
+		(end 109.51 42.4)
+		(stroke
+			(width 0.2)
+			(type solid)
+		)
+		(fill no)
+		(layer "B.SilkS")
+	)
+	(gr_circle
+		(center 46.81 42.4)
+		(end 48.81 42.4)
+		(stroke
+			(width 0.7)
+			(type solid)
+		)
+		(fill no)
+		(layer "B.SilkS")
+	)
+	(gr_circle
+		(center 106.81 114.4)
+		(end 108.81 114.4)
+		(stroke
+			(width 0.7)
+			(type solid)
+		)
+		(fill no)
+		(layer "B.SilkS")
+	)
+	(gr_circle
+		(center 106.81 114.4)
+		(end 109.51 114.4)
+		(stroke
+			(width 0.2)
+			(type solid)
+		)
+		(fill no)
+		(layer "B.SilkS")
+	)
+	(gr_circle
+		(center 46.81 42.4)
+		(end 49.51 42.4)
+		(stroke
+			(width 0.2)
+			(type solid)
+		)
+		(fill no)
+		(layer "B.SilkS")
+	)
+	(gr_circle
+		(center 106.81 42.4)
+		(end 108.81 42.4)
+		(stroke
+			(width 0.7)
+			(type solid)
+		)
+		(fill no)
+		(layer "B.SilkS")
+	)
+	(gr_circle
+		(center 46.81 114.4)
+		(end 49.51 114.4)
+		(stroke
+			(width 0.2)
+			(type solid)
+		)
+		(fill no)
+		(layer "B.SilkS")
+	)
+	(gr_circle
+		(center 46.81 114.4)
+		(end 48.81 114.4)
+		(stroke
+			(width 0.7)
+			(type solid)
+		)
+		(fill no)
+		(layer "B.SilkS")
+	)
+	(gr_circle
 		(center 106.81 114.4)
 		(end 108.31 114.4)
@@
 	)
 	(gr_text "B+"
-		(at 110.22 45.63 90)
+		(at 110.63 46.23 90)
 		(layer "F.SilkS" knockout)
 		(effects
@@
 		)
 	)
-	(gr_text "VUSB"
+	(gr_text "VBUS"
 		(at 108.34 80.06 0)
 		(layer "F.SilkS")
@@
 	)
 	(gr_text "B-"
-		(at 106.1 45.63 90)
+		(at 106.51 46.23 90)
 		(layer "F.SilkS" knockout)
 		(effects
@@
 	)
 	(gr_text "A+"
-		(at 108.846667 45.572857 90)
+		(at 109.256667 46.172857 90)
 		(layer "F.SilkS" knockout)
 		(effects
@@
 	)
 	(gr_text "A-"
-		(at 107.473333 45.572857 90)
+		(at 107.883333 46.172857 90)
 		(layer "F.SilkS" knockout)
 		(effects
@@
 		)
 	)
-	(gr_text "4xM3"
-		(at 46.72 52.56 270)
-		(layer "F.SilkS")
-		(effects
-			(font
-				(size 1.5 1.5)
-				(thickness 0.3)
-				(bold yes)
-			)
-		)
-	)
 	(gr_text "SCL"
 		(at 123.28 106.01 270)
@@
 		(start 103.14 69.54)
 		(end 103.14 77.02)
-		(width 0.4)
+		(width 1)
 		(layer "F.Cu")
 		(net 3)
@@
 		(min_thickness 0.25)
 		(filled_areas_thickness no)
-		(fill
+		(fill yes
 			(thermal_gap 0.5)
 			(thermal_bridge_width 0.5)
@@
 		(min_thickness 0.25)
 		(filled_areas_thickness no)
-		(fill
+		(fill yes
 			(thermal_gap 0.5)
 			(thermal_bridge_width 0.5)
@@
 		(min_thickness 0.25)
 		(filled_areas_thickness no)
-		(fill
+		(fill yes
 			(thermal_gap 0.5)
 			(thermal_bridge_width 0.5)
@@
 		(min_thickness 0.25)
 		(filled_areas_thickness no)
-		(fill
+		(fill yes
 			(thermal_gap 0.5)
 			(thermal_bridge_width 0.5)
@@
 		(min_thickness 0.25)
 		(filled_areas_thickness no)
-		(fill
+		(fill yes
 			(thermal_gap 0.5)
 			(thermal_bridge_width 0.5)
@@
 		(min_thickness 0.25)
 		(filled_areas_thickness no)
-		(fill
+		(fill yes
 			(thermal_gap 0.5)
 			(thermal_bridge_width 0.5)
@@
 		(min_thickness 0.25)
 		(filled_areas_thickness no)
-		(fill
+		(fill yes
 			(thermal_gap 0.5)
 			(thermal_bridge_width 0.5)
@@
 		(min_thickness 0.25)
 		(filled_areas_thickness no)
-		(fill
+		(fill yes
 			(thermal_gap 0.5)
 			(thermal_bridge_width 0.5)
@@
 		(min_thickness 0.25)
 		(filled_areas_thickness no)
-		(fill
+		(fill yes
 			(thermal_gap 0.5)
 			(thermal_bridge_width 0.5)
@@
 		(min_thickness 0.25)
 		(filled_areas_thickness no)
-		(fill
+		(fill yes
 			(thermal_gap 0.5)
 			(thermal_bridge_width 0.5)
@@
 		(min_thickness 0.25)
 		(filled_areas_thickness no)
-		(fill
+		(fill yes
 			(thermal_gap 0.5)
 			(thermal_bridge_width 0.5)
@@
 		(min_thickness 0.25)
 		(filled_areas_thickness no)
-		(fill
+		(fill yes
 			(thermal_gap 0.5)
 			(thermal_bridge_width 0.5)
@@
 		(min_thickness 0.25)
 		(filled_areas_thickness no)
-		(fill
+		(fill yes
 			(thermal_gap 0.5)
 			(thermal_bridge_width 0.5)
@@
 		(min_thickness 0.25)
 		(filled_areas_thickness no)
-		(fill
+		(fill yes
 			(thermal_gap 0.5)
 			(thermal_bridge_width 0.5)
@@
 		(min_thickness 0.25)
 		(filled_areas_thickness no)
-		(fill
+		(fill yes
 			(thermal_gap 0.5)
 			(thermal_bridge_width 0.5)
@@
 		(min_thickness 0.25)
 		(filled_areas_thickness no)
-		(fill
+		(fill yes
 			(thermal_gap 0.5)
 			(thermal_bridge_width 0.5)
@@
 		(min_thickness 0.25)
 		(filled_areas_thickness no)
-		(fill
+		(fill yes
 			(thermal_gap 0.5)
 			(thermal_bridge_width 0.5)
@@
 		(min_thickness 0.25)
 		(filled_areas_thickness no)
-		(fill
+		(fill yes
 			(thermal_gap 0.5)
 			(thermal_bridge_width 0.5)
@@
 		(min_thickness 0.25)
 		(filled_areas_thickness no)
-		(fill
+		(fill yes
 			(thermal_gap 0.5)
 			(thermal_bridge_width 0.5)
@@
 		(min_thickness 0.25)
 		(filled_areas_thickness no)
-		(fill
+		(fill yes
 			(thermal_gap 0.5)
 			(thermal_bridge_width 0.5)
@@
 		(min_thickness 0.25)
 		(filled_areas_thickness no)
-		(fill
+		(fill yes
 			(thermal_gap 0.5)
 			(thermal_bridge_width 0.5)
@@
 		(min_thickness 0.25)
 		(filled_areas_thickness no)
-		(fill
+		(fill yes
 			(thermal_gap 0.5)
 			(thermal_bridge_width 0.5)
@@
 		(min_thickness 0.25)
 		(filled_areas_thickness no)
-		(fill
+		(fill yes
 			(thermal_gap 0.5)
 			(thermal_bridge_width 0.5)
@@
 		(min_thickness 0.25)
 		(filled_areas_thickness no)
-		(fill
+		(fill yes
 			(thermal_gap 0.5)
 			(thermal_bridge_width 0.5)
@@
 		(min_thickness 0.25)
 		(filled_areas_thickness no)
-		(fill
+		(fill yes
 			(thermal_gap 0.5)
 			(thermal_bridge_width 0.5)
@@
 		(min_thickness 0.25)
 		(filled_areas_thickness no)
-		(fill
+		(fill yes
 			(thermal_gap 0.5)
 			(thermal_bridge_width 0.5)
@@
 		(min_thickness 0.25)
 		(filled_areas_thickness no)
-		(fill
+		(fill yes
 			(thermal_gap 0.5)
 			(thermal_bridge_width 0.5)
