File: hardware/DucMinh.kicad_pcb (KiCad board)
At the start: 2 copper layers, 90 x 80 mm, 62 parts, among them J1 Power, J10 HC05, J11 PWR_Selection, J12 BOOT0, J2 M1, J3 USB_B_Micro, J4 M2, J5 M3, J6 AS5600, J7 STLink, J8 Stepper_Motor, SW1 SW_Push, U10 BTS7960B, U2 AMS1117-3.3, U3 LM2596SX-5.0/NOPB, U4 TMC2209_SILENTSTEPSTICK, U5 BTS7960B, U6 STM32F103RCT6, U8 BTS7960B, Y1 8 MHz

Commit message: update
Parts:
- moved R3 11.8 mm to (117.6, 109.7), turned to 0 degrees
- moved C9 0.71 mm to (107.8, 112.9)
Routing:
- net +3V3: track 347.0 -> 326.6 mm
- net Net-(U6-PD0-OSC_IN): track 27.5 -> 26.2 mm
- net Net-(U6-PD1_OSC_OUT): track 21.1 -> 20.2 mm
- net MS1_PIN: track 86.1 -> 85.4 mm
- net ENABLE_PIN: track 89.9 -> 89.2 mm
- net MS2_PIN: track 84.8 -> 84.1 mm

Commit message: a
Other:
- board text added: "SWD"
- board text removed: "STLINK"
Changed lines of the file:
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@@
 	)
 	(gr_text "RX"
-		(at 83.880001 110.65 90)
+		(at 81.125735 110.74 90)
 		(layer "F.SilkS")
 		(effects
@@
 	)
 	(gr_text "TX"
-		(at 86.42 110.65 90)
+		(at 78.585737 110.74 90)
 		(layer "F.SilkS")
 		(effects
@@
 	)
 	(gr_text "GND"
-		(at 81.34 110.65 90)
+		(at 83.665737 110.74 90)
 		(layer "F.SilkS")
 		(effects
@@
 		)
 	)
-	(gr_text "STLINK"
-		(at 127.49 88.27 0)
+	(gr_text "SWD"
+		(at 128.28 88.29 0)
 		(layer "F.SilkS" knockout)
 		(effects
@@
 	)
 	(gr_text "3V3"
-		(at 78.800001 110.65 90)
-		(layer "F.SilkS")
-		(effects
+		(at 86.205736 110.74 90)
+		(layer "F.SilkS")
+		(effects
